File: copy_layout/Destination_project/Destination_project.kicad_pcb (KiCad board)
At the start: 2 copper layers, 11 parts, among them Q1 CSD19531KCS, Q2 CSD19531KCS, U1 LAUNCHXL-F28379D, U2 IR2181, U3 LTS_15

Commit message: Repaired annotation
Connections:
- Q1 pad 3: Net-(Q1-Pad3) -> Net-(C2-Pad1)
- Q2 pad 2: Net-(Q1-Pad3) -> Net-(C2-Pad1)
- R2 pad 1: Net-(C2-Pad1) -> Net-(R2-Pad1)
- U2 pad 4: Net-(C2-Pad1) -> Net-(R2-Pad1)
- U2 pad 6: Net-(U2-Pad6) -> Net-(C2-Pad1)
- U3 pad 1: Net-(Q1-Pad3) -> Net-(C2-Pad1)
- U3 pad 2: Net-(Q1-Pad3) -> Net-(C2-Pad1)
- U3 pad 3: Net-(Q1-Pad3) -> Net-(C2-Pad1)
