File: copy_layout/Destination_project/Leg.sch (KiCad schematic (older format))
At the start: 10 parts, among them Q3 CSD19531KCS, Q4 CSD19531KCS, U4 IR2181, U5 LTS_15

Commit message: Repaired annotation
Parts:
- renumbered C4 to C1, C5 to C2, C6 to C3, D2 to D1, Q3 to Q1, Q4 to Q2, R3 to R1, R4 to R2, U4 to U2, U5 to U3
Connections:
- net at Q1.3 (S), Q2.2 (D), U3.1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: now also C2.1, U2.6 (VS)
- net at R2.1, U2.4 (LO): no longer C2.1
