File: copy_layout/Source_project/Leg.sch (KiCad schematic (older format))
At the start: 10 parts, among them Q3 CSD19531KCS, Q4 CSD19531KCS, U4 IR2181, U5 LTS_15

Commit message: Repaired annotation
Connections:
- net at Q3.3 (S), Q4.2 (D), U5.1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: now also C5.1, U4.6 (VS)
- net at R4.1, U4.4 (LO): no longer C5.1
Changed lines of the file:
@@
 EESchema Schematic File Version 4
+LIBS:Source_project-cache
 EELAYER 29 0
 EELAYER END
 $Descr A4 11693 8268
 encoding utf-8
-Sheet 4 4
+Sheet 2 4
 Title ""
 Date ""
@@
 AR Path="/5CA63F16/5CA6C1F5" Ref="Q3"  Part="1"
 AR Path="/5CA64568/5CA6C1F5" Ref="Q5"  Part="1"
-F 0 "Q5" H 4100 2400 50  0000 L CNN
+AR Path="/5CA3706F/5CA6C1F5" Ref="Q1"  Part="1"
+F 0 "Q1" H 4100 2400 50  0000 L CNN
 F 1 "CSD19531KCS" H 4100 2300 50  0000 L CNN
 F 2 "Discretes:TO-220" H 4100 2200 50  0001 L CNN
@@
 AR Path="/5CA63F16/5CA38D18" Ref="Q4"  Part="1"
 AR Path="/5CA64568/5CA38D18" Ref="Q6"  Part="1"
-F 0 "Q6" H 4100 3300 50  0000 L CNN
+AR Path="/5CA3706F/5CA38D18" Ref="Q2"  Part="1"
+F 0 "Q2" H 4100 3300 50  0000 L CNN
 F 1 "CSD19531KCS" H 4100 3200 50  0000 L CNN
 F 2 "Discretes:TO-220" H 4100 3100 50  0001 L CNN
@@
 AR Path="/5CA63F16/5CA39EA2" Ref="R3"  Part="1"
 AR Path="/5CA64568/5CA39EA2" Ref="R5"  Part="1"
-F 0 "R5" H 3300 2500 50  0000 L CNN
+AR Path="/5CA3706F/5CA39EA2" Ref="R1"  Part="1"
+F 0 "R1" H 3300 2500 50  0000 L CNN
 F 1 "22R" H 3300 2400 50  0000 L CNN
 F 2 "Passives:R1206M" H 3300 2200 50  0001 L CNN
@@
 AR Path="/5CA63F16/5CA3A2D0" Ref="R4"  Part="1"
 AR Path="/5CA64568/5CA3A2D0" Ref="R6"  Part="1"
-F 0 "R6" H 3300 3400 50  0000 L CNN
+AR Path="/5CA3706F/5CA3A2D0" Ref="R2"  Part="1"
+F 0 "R2" H 3300 3400 50  0000 L CNN
 F 1 "22R" H 3300 3300 50  0000 L CNN
 F 2 "Passives:R1206M" H 3300 3100 50  0001 L CNN
@@
 AR Path="/5CA63F16/5CA3CA6D" Ref="U4"  Part="1"
 AR Path="/5CA64568/5CA3CA6D" Ref="U6"  Part="1"
-F 0 "U6" H 2000 3400 50  0000 L CNN
+AR Path="/5CA3706F/5CA3CA6D" Ref="U2"  Part="1"
+F 0 "U2" H 2000 3400 50  0000 L CNN
 F 1 "IR2181" H 2000 3325 50  0000 L CNN
 F 2 "Package_SO:SO8" H 2000 3250 50  0001 L CNN
@@
 Wire Wire Line
 	2500 3000 3100 3000
-Wire Wire Line
-	2500 3200 2750 3200
 $Comp
 L Passives:GND #PWR021
@@
 AR Path="/5CA63F16/5CA3DD1D" Ref="#PWR021"  Part="1"
 AR Path="/5CA64568/5CA3DD1D" Ref="#PWR031"  Part="1"
+AR Path="/5CA3706F/5CA3DD1D" Ref="#PWR011"  Part="1"
 F 0 "#PWR031" H 4000 3500 50  0001 C CNN
 F 1 "GND" H 4150 3600 50  0001 C CNN
@@
 AR Path="/5CA63F16/5CA3E57D" Ref="#PWR019"  Part="1"
 AR Path="/5CA64568/5CA3E57D" Ref="#PWR029"  Part="1"
+AR Path="/5CA3706F/5CA3E57D" Ref="#PWR09"  Part="1"
 F 0 "#PWR029" H 1800 3150 50  0001 C CNN
 F 1 "GND" H 1950 3250 50  0001 C CNN
@@
 AR Path="/5CA63F16/5CA3F09F" Ref="C4"  Part="1"
 AR Path="/5CA64568/5CA3F09F" Ref="C7"  Part="1"
-F 0 "C7" H 1350 2250 50  0000 L CNN
+AR Path="/5CA3706F/5CA3F09F" Ref="C1"  Part="1"
+F 0 "C1" H 1350 2250 50  0000 L CNN
 F 1 "100n" H 1350 2150 50  0000 L CNN
 F 2 "Passives:C1206M" H 1300 2100 50  0001 L CNN
@@
 AR Path="/5CA63F16/5CA40318" Ref="#PWR017"  Part="1"
 AR Path="/5CA64568/5CA40318" Ref="#PWR027"  Part="1"
+AR Path="/5CA3706F/5CA40318" Ref="#PWR07"  Part="1"
 F 0 "#PWR027" H 1250 2250 50  0001 C CNN
 F 1 "GND" H 1400 2350 50  0001 C CNN
@@
 AR Path="/5CA63F16/5CA6C1FE" Ref="#PWR016"  Part="1"
 AR Path="/5CA64568/5CA6C1FE" Ref="#PWR026"  Part="1"
+AR Path="/5CA3706F/5CA6C1FE" Ref="#PWR06"  Part="1"
 F 0 "#PWR026" H 1250 1800 50  0001 C CNN
 F 1 "+12V" H 1250 2090 50  0000 C CNN
@@
 AR Path="/5CA63F16/5CA6C1FF" Ref="#PWR018"  Part="1"
 AR Path="/5CA64568/5CA6C1FF" Ref="#PWR028"  Part="1"
+AR Path="/5CA3706F/5CA6C1FF" Ref="#PWR08"  Part="1"
 F 0 "#PWR028" H 1800 2650 50  0001 C CNN
 F 1 "+12V" H 1800 2940 50  0000 C CNN
@@
 AR Path="/5CA63F16/5CA6C200" Ref="C5"  Part="1"
 AR Path="/5CA64568/5CA6C200" Ref="C8"  Part="1"
-F 0 "C8" H 2850 2150 50  0000 L CNN
+AR Path="/5CA3706F/5CA6C200" Ref="C2"  Part="1"
+F 0 "C2" H 2850 2150 50  0000 L CNN
 F 1 "100n" H 2850 2250 50  0000 L CNN
 F 2 "Passives:C1206M" H 2800 2100 50  0001 L CNN
@@
 AR Path="/5CA63F16/5CA6C201" Ref="D2"  Part="1"
 AR Path="/5CA64568/5CA6C201" Ref="D3"  Part="1"
-F 0 "D3" H 1800 2150 50  0000 L CNN
+AR Path="/5CA3706F/5CA6C201" Ref="D1"  Part="1"
+F 0 "D1" H 1800 2150 50  0000 L CNN
 F 1 "LL4148" H 1650 2250 50  0000 L CNN
 F 2 "Discretes:D_MiniMELF" H 1650 1950 50  0001 L CNN
@@
 	1250 2050 1250 2100
 Wire Wire Line
-	2750 2300 2750 3200
-Connection ~ 2750 3200
-Wire Wire Line
-	2750 3200 3200 3200
-Wire Wire Line
 	2500 2900 2600 2900
 Wire Wire Line
@@
 AR Path="/5CA63F16/5CA6C202" Ref="#PWR020"  Part="1"
 AR Path="/5CA64568/5CA6C202" Ref="#PWR030"  Part="1"
+AR Path="/5CA3706F/5CA6C202" Ref="#PWR010"  Part="1"
 F 0 "#PWR030" H 4000 1800 50  0001 C CNN
 F 1 "+12V" H 4000 2090 50  0000 C CNN
@@
 AR Path="/5CA63F16/5CA51397" Ref="U5"  Part="1"
 AR Path="/5CA64568/5CA51397" Ref="U7"  Part="1"
-F 0 "U7" H 5250 3850 50  0000 L CNN
+AR Path="/5CA3706F/5CA51397" Ref="U3"  Part="1"
+F 0 "U3" H 5250 3850 50  0000 L CNN
 F 1 "LTS_15" H 5250 3750 50  0000 L CNN
 F 2 "Sensor_Current:LTS_15" H 5250 3650 50  0001 L CNN
@@
 AR Path="/5CA63F16/5CA6C204" Ref="#PWR022"  Part="1"
 AR Path="/5CA64568/5CA6C204" Ref="#PWR032"  Part="1"
+AR Path="/5CA3706F/5CA6C204" Ref="#PWR012"  Part="1"
 F 0 "#PWR032" H 4950 2900 50  0001 C CNN
 F 1 "+3.3V" H 4950 3190 50  0000 C CNN
@@
 AR Path="/5CA63F16/5CA573F4" Ref="#PWR023"  Part="1"
 AR Path="/5CA64568/5CA573F4" Ref="#PWR033"  Part="1"
+AR Path="/5CA3706F/5CA573F4" Ref="#PWR013"  Part="1"
 F 0 "#PWR033" H 4950 3200 50  0001 C CNN
 F 1 "GND" H 5100 3300 50  0001 C CNN
@@
 AR Path="/5CA63F16/5CA59426" Ref="#PWR024"  Part="1"
 AR Path="/5CA64568/5CA59426" Ref="#PWR034"  Part="1"
+AR Path="/5CA3706F/5CA59426" Ref="#PWR014"  Part="1"
 F 0 "#PWR034" H 5550 3500 50  0001 C CNN
 F 1 "+3.3V" H 5550 3790 50  0000 C CNN
@@
 AR Path="/5CA63F16/5CA5984D" Ref="#PWR025"  Part="1"
 AR Path="/5CA64568/5CA5984D" Ref="#PWR035"  Part="1"
+AR Path="/5CA3706F/5CA5984D" Ref="#PWR015"  Part="1"
 F 0 "#PWR035" H 5550 3900 50  0001 C CNN
 F 1 "GND" H 5700 4000 50  0001 C CNN
@@
 AR Path="/5CA63F16/5CA59E4B" Ref="C6"  Part="1"
 AR Path="/5CA64568/5CA59E4B" Ref="C9"  Part="1"
-F 0 "C9" H 5650 3800 50  0000 L CNN
+AR Path="/5CA3706F/5CA59E4B" Ref="C3"  Part="1"
+F 0 "C3" H 5650 3800 50  0000 L CNN
 F 1 "100n" H 5650 3900 50  0000 L CNN
 F 2 "Passives:C1206M" H 5600 3750 50  0001 L CNN
@@
 Wire Wire Line
 	5550 3750 5550 3650
+Wire Wire Line
+	2500 3200 3200 3200
+Wire Wire Line
+	2500 3100 2750 3100
+Wire Wire Line
+	2750 3100 2750 2300
+Wire Wire Line
+	4000 2750 3200 2750
+Wire Wire Line
+	3200 2750 3200 3100
+Wire Wire Line
+	3200 3100 2750 3100
+Connection ~ 2750 3100
 $EndSCHEMATC
