File: copy_layout/Source_project/Source_project.kicad_pcb (KiCad board)
At the start: 2 copper layers, 31 parts, among them Q1 CSD19531KCS, Q2 CSD19531KCS, Q3 CSD19531KCS, Q4 CSD19531KCS, Q5 CSD19531KCS, Q6 CSD19531KCS, U1 TMS320F28027PT, U2 IR2181, U3 LTS_15, U4 IR2181, U5 LTS_15, U6 IR2181, U7 LTS_15

Commit message: Repaired annotation
Connections:
- Q3 pad 3: Net-(Q3-Pad3) -> Net-(C5-Pad1)
- Q4 pad 2: Net-(Q3-Pad3) -> Net-(C5-Pad1)
- Q5 pad 3: Net-(Q5-Pad3) -> Net-(C8-Pad1)
- Q6 pad 2: Net-(Q5-Pad3) -> Net-(C8-Pad1)
- R4 pad 1: Net-(C5-Pad1) -> Net-(R4-Pad1)
- R6 pad 1: Net-(C8-Pad1) -> Net-(R6-Pad1)
- U4 pad 4: Net-(C5-Pad1) -> Net-(R4-Pad1)
- U4 pad 6: Net-(U4-Pad6) -> Net-(C5-Pad1)
- U5 pad 1: Net-(Q3-Pad3) -> Net-(C5-Pad1)
- U5 pad 2: Net-(Q3-Pad3) -> Net-(C5-Pad1)
- U5 pad 3: Net-(Q3-Pad3) -> Net-(C5-Pad1)
- U6 pad 4: Net-(C8-Pad1) -> Net-(R6-Pad1)
- U6 pad 6: Net-(U6-Pad6) -> Net-(C8-Pad1)
- U7 pad 1: Net-(Q5-Pad3) -> Net-(C8-Pad1)
- U7 pad 2: Net-(Q5-Pad3) -> Net-(C8-Pad1)
- U7 pad 3: Net-(Q5-Pad3) -> Net-(C8-Pad1)

Commit message: Updated test projects
Routing:
- added copper zone on F.Cu, net Net-(C2-Pad1)
Other:
- board text added: "TEXT"
Changed lines of the file:
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@@
   (general
     (thickness 1.6)
-    (drawings 0)
+    (drawings 1)
     (tracks 48)
     (zones 0)
@@
   )
   (setup
-    (last_trace_width 0.6)
+    (last_trace_width 0.25)
     (user_trace_width 0.4)
     (user_trace_width 0.6)
@@
     (solder_mask_min_width 0.25)
     (aux_axis_origin 0 0)
-    (visible_elements 7FFFFFFF)
+    (visible_elements 7FFFFF7F)
     (pcbplotparams
       (layerselection 0x010fc_ffffffff)
@@
     (tags "SOIC 1.27")
     (attr smd)
-    (fp_text reference U2 (at 0 -3.5 90) (layer F.SilkS)
+    (fp_text reference U2 (at -3.81 -3.81 180) (layer F.SilkS)
       (effects (font (size 1 1) (thickness 0.15)))
     )
@@
     (tags "capacitor 1206")
     (attr smd)
-    (fp_text reference R2 (at 0 -1.75 90) (layer F.SilkS)
+    (fp_text reference R2 (at 0 1.905 180) (layer F.SilkS)
       (effects (font (size 1 1) (thickness 0.15)))
     )
@@
     (tags "capacitor 1206")
     (attr smd)
-    (fp_text reference R1 (at 0 -1.75 90) (layer F.SilkS)
+    (fp_text reference R1 (at 0 1.905 180) (layer F.SilkS)
       (effects (font (size 1 1) (thickness 0.15)))
     )
@@
     (tags "Diode Mini-MELF")
     (attr smd)
-    (fp_text reference D1 (at 0 -2 270) (layer F.SilkS)
+    (fp_text reference D1 (at -3.81 0.635) (layer F.SilkS)
       (effects (font (size 1 1) (thickness 0.15)))
     )
@@
     (tags "capacitor 1206")
     (attr smd)
-    (fp_text reference C2 (at 0 -1.75 180) (layer F.SilkS)
+    (fp_text reference C2 (at 0 1.905 180) (layer F.SilkS)
       (effects (font (size 1 1) (thickness 0.15)))
     )
@@
     (tags "capacitor 1206")
     (attr smd)
-    (fp_text reference C1 (at 0 -1.75) (layer F.SilkS)
+    (fp_text reference C1 (at 0 1.905) (layer F.SilkS)
       (effects (font (size 1 1) (thickness 0.15)))
     )
@@
     )
   )
+  (gr_text TEXT (at 180.34 63.5) (layer F.SilkS)
+    (effects (font (size 1 1) (thickness 0.15)))
+  )
   (segment (start 172.085 74.525) (end 171.68 74.93) (width 0.6) (layer F.Cu) (net 1))
   (segment (start 172.085 71.915) (end 172.085 74.525) (width 0.6) (layer F.Cu) (net 1))
@@
   (segment (start 172.085 63.73) (end 172.315 63.5) (width 0.6) (layer F.Cu) (net 4))
   (segment (start 172.085 66.515) (end 172.085 63.73) (width 0.6) (layer F.Cu) (net 4))
+  (segment (start 167.41 34.29) (end 167.64 34.06) (width 0.6) (layer B.Cu) (net 5))
+  (segment (start 165.1 34.29) (end 167.41 34.29) (width 0.6) (layer B.Cu) (net 5))
   (segment (start 165.1 50.8) (end 165.1 55.65) (width 1) (layer F.Cu) (net 10))
   (segment (start 177.878 55.572) (end 177.8 55.65) (width 1) (layer F.Cu) (net 11))
@@
   (segment (start 177.8 68.37) (end 174.255 71.915) (width 0.6) (layer F.Cu) (net 64))
   (segment (start 177.8 58.65) (end 177.8 68.37) (width 0.6) (layer F.Cu) (net 64))
-  (segment (start 167.41 34.29) (end 167.64 34.06) (width 0.6) (layer B.Cu) (net 5))
-  (segment (start 165.1 34.29) (end 167.41 34.29) (width 0.6) (layer B.Cu) (net 5))
+  (zone (net 4) (net_name "Net-(C2-Pad1)") (layer F.Cu) (hatch edge 0.508)
+    (connect_pads yes (clearance 0.508))
+    (min_thickness 0.254)
+    (fill yes (arc_segments 32) (thermal_gap 0.508) (thermal_bridge_width 0.508))
+    (polygon
+      (pts
+        (xy 169.545 41.275) (xy 181.61 41.275) (xy 181.61 52.07) (xy 168.91 52.07) (xy 168.91 41.275)
+      )
+    )
+  )
 )
